Commit message: use xacro for variable path

File: rover_description/urdf/urdf_wheel.urdf (robot description, URDF)
Before this commit: robot rover_description, 5 links, 4 joints
Links:
- link base_link: geometry collision mesh filename=$(arg rover_path)/meshes/base_link.STL; visual mesh filename=$(arg rover_path)/meshes/base_link.STL
- link joint_1: geometry collision mesh filename=$(arg rover_path)/meshes/joint_1.STL; visual mesh filename=$(arg rover_path)/meshes/joint_1.STL
- link joint_2: geometry collision mesh filename=$(arg rover_path)/meshes/joint_2.STL; visual mesh filename=$(arg rover_path)/meshes/joint_2.STL
- link joint_3: geometry collision mesh filename=$(arg rover_path)/meshes/joint_3.STL; visual mesh filename=$(arg rover_path)/meshes/joint_3.STL
- link joint_4: geometry collision mesh filename=$(arg rover_path)/meshes/joint_4.STL; visual mesh filename=$(arg rover_path)/meshes/joint_4.STL

Commit message: fix for rviz path resolve problem

File: rover_description/urdf/urdf_wheel.urdf (robot description, URDF)
Before this commit: robot rover_description, 5 links, 4 joints
Links:
- link base_link: geometry collision mesh filename=file://$(arg rover_path)/meshes/base_link.STL; visual mesh filename=file://$(arg rover_path)/meshes/base_link.STL
- link joint_1: geometry collision mesh filename=file://$(arg rover_path)/meshes/joint_1.STL; visual mesh filename=file://$(arg rover_path)/meshes/joint_1.STL
- link joint_2: geometry collision mesh filename=file://$(arg rover_path)/meshes/joint_2.STL; visual mesh filename=file://$(arg rover_path)/meshes/joint_2.STL
- link joint_3: geometry collision mesh filename=file://$(arg rover_path)/meshes/joint_3.STL; visual mesh filename=file://$(arg rover_path)/meshes/joint_3.STL
- link joint_4: geometry collision mesh filename=file://$(arg rover_path)/meshes/joint_4.STL; visual mesh filename=file://$(arg rover_path)/meshes/joint_4.STL

Commit message: new body

File: rover_description/urdf/urdf_wheel.urdf (robot description, URDF)
Before this commit: robot rover_description, 5 links, 4 joints
Links:
- link base_link: mass 18.9097180944353 -> 18.2799897993079
Joints:
- joint wheel_4: origin xyz=-0.412250550889761 -0.349292562707965 -0.387276310870224 rpy=3.14159265358979 0 3.14159265358979 -> xyz=-0.41225 -0.34929 -0.38728 rpy=3.1416 0 3.1416

Commit message: bug fix: urdf rotational axis fix

File: rover_description/urdf/urdf_wheel.urdf (robot description, URDF)
Before this commit: robot rover_description, 5 links, 4 joints
Joints:
- joint wheel_1: axis -1 0 0 -> 1 0 0
- joint wheel_4: axis -1 0 0 -> 1 0 0

Commit message: new urdf: chnaged axis

File: rover_description/urdf/urdf_wheel.urdf (robot description, URDF)
Before this commit: robot rover_description, 5 links, 4 joints
Links:
- link base_link: mass 18.2799897993079 -> 18.9097180944353
- link joint_3: mass 0.978512007649862 -> 0.978511891131766
- link joint_4: mass 0.978512007561894 -> 0.97851190354741
Joints:
- joint wheel_1: axis 1 0 0 -> 0 -1 0; origin xyz=-0.41211 0.39068 -0.38728 rpy=3.1416 0 3.1416 -> xyz=-0.41211 0.39068 -0.38728 rpy=0 0 -1.5707963267949
- joint wheel_2: axis 1 0 0 -> 0 -1 0; origin xyz=0.37451 0.39068 -0.38728 rpy=3.1416 0 3.1416 -> xyz=0.374505 0.39068 -0.38726 rpy=0 0 -1.5708
- joint wheel_3: axis 1 0 0 -> 0 -1 0; origin xyz=0.37465 -0.34929 -0.38728 rpy=3.1416 0 3.1416 -> xyz=0.37465 -0.34929 -0.38728 rpy=0 0 -1.57079
- joint wheel_4: axis 1 0 0 -> 0 -1 0; origin xyz=-0.41225 -0.34929 -0.38728 rpy=3.1416 0 3.1416 -> xyz=-0.41225 -0.34929 -0.38728 rpy=0 0 -1.5707963267949

Commit message: new urdf body rotated

File: rover_description/urdf/urdf_wheel.urdf (robot description, URDF)
Before this commit: robot rover_description, 5 links, 4 joints
Joints:
- joint wheel_1: axis 0 -1 0 -> 0 1 0; origin xyz=-0.41211 0.39068 -0.38728 rpy=0 0 -1.5707963267949 -> xyz=-0.39068 -0.41211 -0.38728 rpy=0 0 0
- joint wheel_2: axis 0 -1 0 -> 0 1 0; origin xyz=0.374505 0.39068 -0.38726 rpy=0 0 -1.5708 -> xyz=-0.390678841233882 0.374505301267686 -0.387276310870224 rpy=0 0 0
- joint wheel_3: axis 0 -1 0 -> 0 1 0; origin xyz=0.37465 -0.34929 -0.38728 rpy=0 0 -1.57079 -> xyz=0.349292562707965 0.374648069983417 -0.387276310870224 rpy=0 0 0
- joint wheel_4: axis 0 -1 0 -> 0 1 0; origin xyz=-0.41225 -0.34929 -0.38728 rpy=0 0 -1.5707963267949 -> xyz=0.349292562707965 -0.412250550889761 -0.387276310870224 rpy=0 0 0

Commit message: some how fixed the visual

File: rover_description/urdf/urdf_wheel.urdf (robot description, URDF)
Before this commit: robot rover_description, 5 links, 4 joints
Joints:
- joint wheel_1: origin xyz=-0.39068 -0.41211 -0.38728 rpy=0 0 0 -> xyz=0.349292562707965 0.374648069983417 -0.387276310870224 rpy=0 0 0
- joint wheel_2: origin xyz=-0.390678841233882 0.374505301267686 -0.387276310870224 rpy=0 0 0 -> xyz=0.349292562707965 -0.412250550889761 -0.387276310870224 rpy=0 0 0
- joint wheel_3: origin xyz=0.349292562707965 0.374648069983417 -0.387276310870224 rpy=0 0 0 -> xyz=-0.39068 -0.41211 -0.38728 rpy=0 0 0
- joint wheel_4: origin xyz=0.349292562707965 -0.412250550889761 -0.387276310870224 rpy=0 0 0 -> xyz=-0.390678841233882 0.374505301267686 -0.387276310870224 rpy=0 0 0

Commit message: head back to previous urdf

File: rover_description/urdf/urdf_wheel.urdf (robot description, URDF)
Before this commit: robot rover_description, 5 links, 4 joints
Joints:
- joint wheel_1: origin xyz=0.349292562707965 0.374648069983417 -0.387276310870224 rpy=0 0 0 -> xyz=-0.39068 -0.41211 -0.38728 rpy=0 0 0
- joint wheel_2: origin xyz=0.349292562707965 -0.412250550889761 -0.387276310870224 rpy=0 0 0 -> xyz=-0.390678841233882 0.374505301267686 -0.387276310870224 rpy=0 0 0
- joint wheel_3: origin xyz=-0.39068 -0.41211 -0.38728 rpy=0 0 0 -> xyz=0.349292562707965 0.374648069983417 -0.387276310870224 rpy=0 0 0
- joint wheel_4: origin xyz=-0.390678841233882 0.374505301267686 -0.387276310870224 rpy=0 0 0 -> xyz=0.349292562707965 -0.412250550889761 -0.387276310870224 rpy=0 0 0

Commit message: current urdf won't work without this rotational axis

File: rover_description/urdf/urdf_wheel.urdf (robot description, URDF)
Before this commit: robot rover_description, 5 links, 4 joints
Joints:
- joint wheel_1: axis 0 1 0 -> 0 -1 0
- joint wheel_2: axis 0 1 0 -> 0 -1 0
- joint wheel_3: axis 0 1 0 -> 0 -1 0
- joint wheel_4: axis 0 1 0 -> 0 -1 0

Commit message: manually urdf created

File: rover_description/urdf/urdf_wheel.urdf (robot description, URDF)
Before this commit: robot rover_description, 5 links, 4 joints
Links:
- removed link joint_1
- removed link joint_2
- removed link joint_3
- removed link joint_4
- added link BL_wheel; collision mesh filename=file:///mnt/d/coding/urdf_ws/install/rover_description/shar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; visual mesh filename=file:///mnt/d/coding/urdf_ws/install/rover_description/shar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
- added link BR_wheel; collision mesh filename=file:///mnt/d/coding/urdf_ws/install/rover_description/shar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; visual mesh filename=file:///mnt/d/coding/urdf_ws/install/rover_description/shar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
- added link FL_wheel; collision mesh filename=file:///mnt/d/coding/urdf_ws/install/rover_description/shar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; visual mesh filename=file:///mnt/d/coding/urdf_ws/install/rover_description/shar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
- added link FR_wheel; collision mesh filename=file:///mnt/d/coding/urdf_ws/install/rover_description/shar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; visual mesh filename=file:///mnt/d/coding/urdf_ws/install/rover_description/shar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
- link base_link: mass 18.9097180944353 -> None; geometry collision mesh filename=file:///mnt/d/coding/urdf_ws/install/rover_description/shar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; visual mesh filename=file:///mnt/d/coding/urdf_ws/install/rover_description/shar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
Joints:
- removed joint wheel_1
- removed joint wheel_2
- removed joint wheel_3
- removed joint wheel_4
- added joint BL_joint: type continuous, parent base_link, child BL_wheel, origin xyz=-0.385612 0.413443 0.131906 rpy=0 0 0, axis 0 1 0, limit effort=20 velocity=20
- added joint BR_joint: type continuous, parent base_link, child BR_wheel, origin xyz=-0.377044 -0.421409 0.132084 rpy=0 0 0, axis 0 1 0, limit effort=20 velocity=20
- added joint FL_joint: type continuous, parent base_link, child FL_wheel, origin xyz=0.359424 0.412712 0.132259 rpy=0 0 0, axis 0 1 0, limit effort=20 velocity=20
- added joint FR_joint: type continuous, parent base_link, child FR_wheel, origin xyz=0.357788 -0.421409 0.132618 rpy=0 0 0, axis 0 1 0, limit effort=20 velocity=20

Commit message: base footprint added

File: rover_description/urdf/urdf_wheel.urdf (robot description, URDF)
Before this commit: robot rover_description, 5 links, 4 joints
Links:
- added link base_footprint
Joints:
- added joint base_footprint_joint: type fixed, parent base_footprint, child base_link, origin xyz=0 0 .52019 rpy=0 0 0
- joint BL_joint: origin xyz=-0.385612 0.413443 0.131906 rpy=0 0 0 -> xyz=-0.385612 0.413443 -0.386925 rpy=0 0 0
- joint BR_joint: origin xyz=-0.377044 -0.421409 0.132084 rpy=0 0 0 -> xyz=-0.377044 -0.421409 -0.383722 rpy=0 0 0
- joint FL_joint: origin xyz=0.359424 0.412712 0.132259 rpy=0 0 0 -> xyz=0.359424 0.412712 -0.386553 rpy=0 0 0
- joint FR_joint: origin xyz=0.357788 -0.421409 0.132618 rpy=0 0 0 -> xyz=0.357788 -0.421409 -0.387336 rpy=0 0 0

Commit message: innertia added for gazebo

File: rover_description/urdf/urdf_wheel.urdf (robot description, URDF)
Before this commit: robot rover_description, 6 links, 5 joints
Links:
- link BL_wheel: mass None -> 0.95177
- link BR_wheel: mass None -> 0.95177
- link FL_wheel: mass None -> 0.95177
- link FR_wheel: mass None -> 0.95177
- link base_link: mass None -> 18.186723515946

Commit message: dynamic path from launch file

File: rover_description/urdf/urdf_wheel.urdf (robot description, URDF)
Before this commit: robot rover_description, 6 links, 5 joints
Links:
- link BL_wheel: geometry collision mesh filename=file://$(arg rover_path)/meshes/left_wheel.stl; visual mesh filename=file://$(arg rover_path)/meshes/left_wheel.stl
- link BR_wheel: geometry collision mesh filename=file://$(arg rover_path)/meshes/right_wheel.stl; visual mesh filename=file://$(arg rover_path)/meshes/right_wheel.stl
- link FL_wheel: geometry collision mesh filename=file://$(arg rover_path)/meshes/left_wheel.stl; visual mesh filename=file://$(arg rover_path)/meshes/left_wheel.stl
- link FR_wheel: geometry collision mesh filename=file://$(arg rover_path)/meshes/right_wheel.stl; visual mesh filename=file://$(arg rover_path)/meshes/right_wheel.stl
- link base_link: geometry collision mesh filename=file://$(arg rover_path)/meshes/robot_base.stl; visual mesh filename=file://$(arg rover_path)/meshes/robot_base.stl
