Commit message: bugfix: rtab_map not received any data

File: rover_description/urdf/camera_sensor.xacro (robot description, xacro)
@@ -5,4 +5,9 @@
         <parent link="base_link" />
         <child link="camera_sensor" />
+        <!-- rpy is adjusted for rtabmap  -->
+        <!-- blue -> foward
+        red -> up
+        green -> left -->
+        <!-- <origin xyz=".1 .1 .1" rpy="3.14159 -1.5708 0"/> -->
         <origin xyz=".1 .1 .1" rpy="0 0 0"/>
     </joint>
