Commit message: imu: pos & refreash rate

File: rover_description/urdf/imu_sensor.xacro (robot description, xacro)
@@ -5,10 +5,10 @@
         <parent link="base_link" />
         <child link="imu_sensor" />
-        <origin xyz="0 0 0" rpy="0 0 0"/>
+        <origin xyz="0 0 .1" rpy="0 0 0"/>
     </joint>
     <gazebo reference="imu_sensor">
         <sensor name="imu_sensor" type="imu">
             <always_on>1</always_on>
-            <update_rate>1</update_rate>
+            <update_rate>.25</update_rate>
             <visualize>true</visualize>
             <topic>imu</topic>

Commit message: imu orientation reference frame

File: rover_description/urdf/imu_sensor.xacro (robot description, xacro)
@@ -2,4 +2,5 @@
 <robot xmlns:xacro="http://www.ros.org/wiki/xacro">
     <link name="imu_sensor"/>
+    <!-- </link> -->
     <joint name="imu_sensor_joint" type="fixed">
         <parent link="base_link" />
@@ -10,7 +11,15 @@
         <sensor name="imu_sensor" type="imu">
             <always_on>1</always_on>
-            <update_rate>.25</update_rate>
+            <update_rate>1</update_rate>
             <visualize>true</visualize>
             <topic>imu</topic>
+            <imu>
+                <orientation_reference_frame>
+                    <localization>CUSTOM</localization>
+                    <custom_rpy parent_frame='base_link'>
+                    0 0 0
+                    </custom_rpy>
+                </orientation_reference_frame>
+            </imu>
         </sensor>
     </gazebo>

Commit message: update frequency

File: rover_description/urdf/imu_sensor.xacro (robot description, xacro)
@@ -2,5 +2,4 @@
 <robot xmlns:xacro="http://www.ros.org/wiki/xacro">
     <link name="imu_sensor"/>
-    <!-- </link> -->
     <joint name="imu_sensor_joint" type="fixed">
         <parent link="base_link" />
@@ -11,5 +10,6 @@
         <sensor name="imu_sensor" type="imu">
             <always_on>1</always_on>
-            <update_rate>1</update_rate>
+            <update_rate>20</update_rate>
+            <!-- to fule it should be same rate as camera -->
             <visualize>true</visualize>
             <topic>imu</topic>
